Commit message: rename

File: urdf/fixed_camera.urdf.xacro (robot description, xacro)
@@ -1,33 +1,28 @@
 <?xml version="1.0"?>
-<robot name="webcam" xmlns:xacro="http://www.ros.org/wiki/xacro">
-  <!-- Lidar sensors -->
-  <xacro:property name="webcam_size" value="0.050" /> <!-- in m -->
-  <xacro:property name="webcam_mass" value="0.160" /> <!-- in kg-->
-  <xacro:macro name="webcam" params="sub parent transX transY transZ">
-    <!-- sub: l,r 0,1,2,3 etc -->
-    <!-- parent: parent link name -->
-    <!-- transX transY transZ: xyz position -->
-    <link name="webcam_${sub}">
+<robot name="fixed_camera" xmlns:xacro="http://www.ros.org/wiki/xacro">
+  <xacro:property name="camera_size" value="0.05" />
+  <xacro:macro name="fixed_camera" params="number parent transX transY transZ">
+    <link name="camera_${number}">
       <visual>
         <origin xyz="0 0 0" rpy="0 0 0" />
         <geometry>
-          <box size="${webcam_size} ${webcam_size} ${webcam_size}" />
+          <box size="${camera_size} ${camera_size} ${camera_size}" />
         </geometry>
         <material name="Green" />
       </visual>
     </link>
-    <joint name="webcam_${sub}_joint" type="fixed">
+    <joint name="camera_${number}_joint" type="fixed">
       <origin xyz="${transX} ${transY} ${transZ}" rpy="0 0 0" />
       <parent link="${parent}"/>
-      <child link="webcam_${sub}"/>
+      <child link="camera_${number}"/>
     </joint>
-    <gazebo reference="webcam_${sub}">
+    <gazebo reference="camera_${number}">
       <material>Gazebo/Green</material>
       <visualize>true</visualize>
       <turnGravityOff>true</turnGravityOff>
-      <sensor type="camera" name="webcam_${sub}_camera">
+      <sensor type="camera" name="camera_${number}_camera">
         <update_rate>10.0</update_rate>
-        <camera name="webcam_${sub}_camera">
-          <pose>${webcam_size/2} 0 0 0 0 0}</pose>
+        <camera name="camera_${number}_camera">
+          <pose>${camera_size/2} 0 0 0 0 0}</pose>
           <horizontal_fov>1.3962634</horizontal_fov>
           <image>
@@ -49,8 +44,8 @@
           <alwaysOn>true</alwaysOn>
           <updateRate>0.0</updateRate>
-          <cameraName>webcam_${sub}_camera</cameraName>
+          <cameraName>camera_${number}_camera</cameraName>
           <imageTopicName>image_raw</imageTopicName>
           <cameraInfoTopicName>camera_info</cameraInfoTopicName>
-          <frameName>webcam_${sub}</frameName>
+          <frameName>camera_${number}</frameName>
           <hackBaseline>0.0</hackBaseline>
           <distortionK1>0.0</distortionK1>

File: urdf/top_cam.urdf.xacro (robot description, xacro)
@@ -1,8 +1,8 @@
 <?xml version="1.0"?>
 <robot name="top_cam" xmlns:xacro="http://www.ros.org/wiki/xacro">
-  <!-- Included URDF/XACRO Files -->
-  <xacro:include filename="$(find cbot)/urdf/common.urdf.xacro" />
-  <xacro:include filename="$(find cbot)/urdf/webcam.urdf.xacro" />
-  <!-- base_footprint Definition -->
+  <xacro:include filename="$(find top_cam)/urdf/common.urdf.xacro" />
+  <xacro:include filename="$(find top_cam)/urdf/fixed_camera.urdf.xacro" />
+  <!-- for gazebo requirement -->
+  <!-- https://classic.gazebosim.org/tutorials?tut=ros_urdf&cat=connect_ros -->
   <link name="world" />
   <!-- base Definition -->
@@ -11,12 +11,12 @@
     <visual>
       <geometry>
-        <box size="0.03 0.03 0.050"/>
+        <box size="0.03 0.03 0.03"/>
       </geometry>
       <material name="White" />
     </visual>
     <inertial>
-      <mass value="0.2" />
+      <mass value="0.1" />
       <origin xyz="0 0 0" rpy="0 0 0" />
-      <xacro:box_inertia m="0.2" x="0.069" y="0.138" z="0.050" />
+      <xacro:box_inertia m="0.1" x="0.01" y="0.01" z="0.01" />
     </inertial>
   </link>
@@ -26,10 +26,10 @@
   </gazebo>
   <joint name="base_joint" type="fixed">
-    <origin xyz="0 0 0.045" rpy="0 0 0" />
+    <origin xyz="0 0 0" rpy="0 0 0" />
     <parent link="world" />
     <child  link="base_link" />
   </joint>
   <!-- Camera Definition -->
-  <xacro:webcam sub="0" parent="base_link"
+  <xacro:fixed_camera number="0" parent="base_link"
     transX="0" transY="0" transZ="3.0" />
 </robot>

Commit message: CR delete

File: urdf/fixed_camera.urdf.xacro (robot description, xacro)
@@ -2,5 +2,5 @@
 <robot name="fixed_camera" xmlns:xacro="http://www.ros.org/wiki/xacro">
   <xacro:property name="camera_size" value="0.05" />
-  <xacro:macro name="fixed_camera" params="number parent transX transY transZ">
+  <xacro:macro name="fixed_camera" params="number parent transX transY transZ roll pitch yaw">
     <link name="camera_${number}">
       <visual>
@@ -13,5 +13,5 @@
     </link>
     <joint name="camera_${number}_joint" type="fixed">
-      <origin xyz="${transX} ${transY} ${transZ}" rpy="0 0 0" />
+      <origin xyz="${transX} ${transY} ${transZ}" rpy="${roll} ${pitch} ${yaw}" />
       <parent link="${parent}"/>
       <child link="camera_${number}"/>
@@ -21,9 +21,9 @@
       <visualize>true</visualize>
       <turnGravityOff>true</turnGravityOff>
-      <sensor type="camera" name="camera_${number}_camera">
+      <sensor type="camera" name="camera_${number}">
         <update_rate>10.0</update_rate>
-        <camera name="camera_${number}_camera">
+        <camera name="camera_${number}">
           <pose>${camera_size/2} 0 0 0 0 0}</pose>
-          <horizontal_fov>1.3962634</horizontal_fov>
+          <horizontal_fov>1.6</horizontal_fov><!--larger:wide-vier smaller:shallow-->
           <image>
             <width>800</width>
@@ -44,5 +44,5 @@
           <alwaysOn>true</alwaysOn>
           <updateRate>0.0</updateRate>
-          <cameraName>camera_${number}_camera</cameraName>
+          <cameraName>camera_${number}</cameraName>
           <imageTopicName>image_raw</imageTopicName>
           <cameraInfoTopicName>camera_info</cameraInfoTopicName>

File: urdf/top_cam.urdf.xacro (robot description, xacro)
@@ -32,6 +32,6 @@
   <!-- camera link -->
   <xacro:fixed_camera number="0" parent="base_link"
-    transX="0" transY="0" transZ="3.0" />
+    transX="0" transY="0" transZ="4.0" roll="0.0" pitch="1.57" yaw="0.0" />
   <xacro:fixed_camera number="1" parent="base_link"
-    transX="0" transY="1.0" transZ="2.0" />
+    transX="0" transY="1.0" transZ="3.0" roll="0.0" pitch="1.57" yaw="0.0"/>
 </robot>
